File: techweekpcb/drive.kicad_sch (KiCad schematic)
At the start: 1 part

Commit message: Routing and Nerokas BOM
Parts:
- removed J6: ~, Connector_PinHeader_2.54mm:PinHeader_1x06_P2.54mm_Vertical, symbol Connector:Conn_01x06_Male
- added J2: Conn_01x07_Male, Connector_PinHeader_2.54mm:PinHeader_1x07_P2.54mm_Vertical, symbol Connector:Conn_01x07_Male
Connections:
- net ENA: now also J2.1 (Pin_1)
- net ENB: now also J2.7 (Pin_7)
- net IN1: now also J2.2 (Pin_2)
- net IN2: now also J2.3 (Pin_3)
- net IN3: now also J2.5 (Pin_5)
- net IN4: now also J2.6 (Pin_6)
- new net GND: J2.4 (Pin_4)
Changed lines of the file:
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@@
     (stroke (width 0) (type default) (color 0 0 0 0))
   )
-  (wire (pts (xy 101.6 63.5) (xy 105.41 63.5))
+  (wire (pts (xy 116.84 63.5) (xy 116.84 72.39))
+    (stroke (width 0) (type default) (color 0 0 0 0))
+  )
+  (wire (pts (xy 101.6 71.12) (xy 105.41 71.12))
+    (stroke (width 0) (type default) (color 0 0 0 0))
+  )
+  (wire (pts (xy 101.6 60.96) (xy 105.41 60.96))
     (stroke (width 0) (type default) (color 0 0 0 0))
   )
@@
     (stroke (width 0) (type default) (color 0 0 0 0))
   )
-  (wire (pts (xy 105.41 60.96) (xy 101.6 60.96))
+  (wire (pts (xy 101.6 63.5) (xy 116.84 63.5))
     (stroke (width 0) (type default) (color 0 0 0 0))
   )
@@
     )
   )
-  (global_label "IN3" (shape input) (at 105.41 63.5 0) (fields_autoplaced)
+  (global_label "IN3" (shape input) (at 105.41 66.04 0) (fields_autoplaced)
     (effects (font (size 1.27 1.27)) (justify left))
-    (property "Intersheet References" "${INTERSHEET_REFS}" (id 0) (at 110.9679 63.4206 0)
+    (property "Intersheet References" "${INTERSHEET_REFS}" (id 0) (at 110.9679 65.9606 0)
       (effects (font (size 1.27 1.27)) (justify left) hide)
     )
   )
-  (global_label "ENB" (shape input) (at 105.41 68.58 0) (fields_autoplaced)
+  (global_label "ENB" (shape input) (at 105.41 71.12 0) (fields_autoplaced)
     (effects (font (size 1.27 1.27)) (justify left))
-    (property "Intersheet References" "${INTERSHEET_REFS}" (id 0) (at 111.5726 68.5006 0)
+    (property "Intersheet References" "${INTERSHEET_REFS}" (id 0) (at 111.5726 71.0406 0)
       (effects (font (size 1.27 1.27)) (justify left) hide)
     )
@@
     )
   )
-  (global_label "IN4" (shape input) (at 105.41 66.04 0) (fields_autoplaced)
+  (global_label "IN4" (shape input) (at 105.41 68.58 0) (fields_autoplaced)
     (effects (font (size 1.27 1.27)) (justify left))
-    (property "Intersheet References" "${INTERSHEET_REFS}" (id 0) (at 110.9679 65.9606 0)
+    (property "Intersheet References" "${INTERSHEET_REFS}" (id 0) (at 110.9679 68.5006 0)
       (effects (font (size 1.27 1.27)) (justify left) hide)
     )
   )
-  (symbol (lib_id "Connector:Conn_01x06_Male") (at 96.52 60.96 0) (unit 1)
+  (symbol (lib_id "Connector:Conn_01x07_Male") (at 96.52 63.5 0) (unit 1)
     (in_bom yes) (on_board yes) (fields_autoplaced)
-    (property "Reference" "J6" (id 0) (at 97.155 50.8 0))
-    (property "Value" "~" (id 1) (at 97.155 53.34 0))
-    (property "Footprint" "Connector_PinHeader_2.54mm:PinHeader_1x06_P2.54mm_Vertical" (id 2) (at 96.52 60.96 0)
+    (property "Reference" "J2" (id 0) (at 97.155 50.8 0))
+    (property "Value" "Conn_01x07_Male" (id 1) (at 97.155 53.34 0))
+    (property "Footprint" "Connector_PinHeader_2.54mm:PinHeader_1x07_P2.54mm_Vertical" (id 2) (at 96.52 63.5 0)
       (effects (font (size 1.27 1.27)) hide)
     )
-    (property "Datasheet" "~" (id 3) (at 96.52 60.96 0)
-      (effects (font (size 1.27 1.27)) hide)
-    )
-    (property "Nerokas link" "https://store.nerokas.co.ke/index.php?route=product/product&product_id=107" (id 4) (at 96.52 60.96 0)
+    (property "Datasheet" "~" (id 3) (at 96.52 63.5 0)
       (effects (font (size 1.27 1.27)) hide)
     )
@@
     (pin "5")
     (pin "6")
+    (pin "7")
+  )
+  (symbol (lib_id "power:GND") (at 116.84 72.39 0) (unit 1)
+    (in_bom yes) (on_board yes) (fields_autoplaced)
+    (property "Reference" "#PWR0119" (id 0) (at 116.84 78.74 0)
+      (effects (font (size 1.27 1.27)) hide)
+    )
+    (property "Value" "GND" (id 1) (at 116.84 77.47 0))
+    (property "Footprint" "" (id 2) (at 116.84 72.39 0)
+      (effects (font (size 1.27 1.27)) hide)
+    )
+    (property "Datasheet" "" (id 3) (at 116.84 72.39 0)
+      (effects (font (size 1.27 1.27)) hide)
+    )
+    (pin "1")
   )
 )
