File: techweekpcb/indicators.kicad_sch (KiCad schematic)
At the start: 8 parts

Commit message: Routing and Nerokas BOM
Parts:
- removed D1, D2: LED, LED_THT:LED_D5.0mm, symbol Device:LED
- removed R14, R15: 100, UserLibrary:R_Axial_DIN0207_L6.3mm_D2.5mm_P10.16mm_Horizontal, symbol Device:R_Small
Connections:
- net HLIGHT1 renamed RLIGHT3
- net RLIGHT3: no longer R17.1
- new net RLIGHT4: R17.1
Changed lines of the file:
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@@
-    (stroke (width 0) (type default) (color 0 0 0 0))
-  )
-  (wire (pts (xy 110.49 46.99) (xy 114.3 46.99))
     (stroke (width 0) (type default) (color 0 0 0 0))
   )
@@
     (stroke (width 0) (type default) (color 0 0 0 0))
   )
-  (wire (pts (xy 101.6 46.99) (xy 102.87 46.99))
-    (stroke (width 0) (type default) (color 0 0 0 0))
-  )
-  (wire (pts (xy 71.12 46.99) (xy 74.93 46.99))
-    (stroke (width 0) (type default) (color 0 0 0 0))
-  )
   (wire (pts (xy 137.16 46.99) (xy 138.43 46.99))
     (stroke (width 0) (type default) (color 0 0 0 0))
   )
-  (wire (pts (xy 62.23 46.99) (xy 63.5 46.99))
-    (stroke (width 0) (type default) (color 0 0 0 0))
-  )
   (wire (pts (xy 170.18 46.99) (xy 171.45 46.99))
-    (stroke (width 0) (type default) (color 0 0 0 0))
-  )
-  (wire (pts (xy 55.88 46.99) (xy 57.15 46.99))
-    (stroke (width 0) (type default) (color 0 0 0 0))
-  )
-  (wire (pts (xy 114.3 46.99) (xy 114.3 57.15))
-    (stroke (width 0) (type default) (color 0 0 0 0))
-  )
-  (wire (pts (xy 95.25 46.99) (xy 96.52 46.99))
     (stroke (width 0) (type default) (color 0 0 0 0))
   )
@@
     (stroke (width 0) (type default) (color 0 0 0 0))
   )
-  (wire (pts (xy 74.93 46.99) (xy 74.93 57.15))
-    (stroke (width 0) (type default) (color 0 0 0 0))
-  )
-  (global_label "HLIGHT1" (shape input) (at 130.81 46.99 180) (fields_autoplaced)
+  (global_label "RLIGHT3" (shape input) (at 130.81 46.99 180) (fields_autoplaced)
     (effects (font (size 1.27 1.27)) (justify right))
-    (property "Intersheet References" "${INTERSHEET_REFS}" (id 0) (at 120.6559 46.9106 0)
+    (property "Intersheet References" "${INTERSHEET_REFS}" (id 0) (at 120.7164 46.9106 0)
       (effects (font (size 1.27 1.27)) (justify right) hide)
     )
   )
-  (global_label "HLIGHT1" (shape input) (at 55.88 46.99 180) (fields_autoplaced)
+  (global_label "RLIGHT4" (shape input) (at 163.83 46.99 180) (fields_autoplaced)
     (effects (font (size 1.27 1.27)) (justify right))
-    (property "Intersheet References" "${INTERSHEET_REFS}" (id 0) (at 45.7259 46.9106 0)
+    (property "Intersheet References" "${INTERSHEET_REFS}" (id 0) (at 153.7364 46.9106 0)
       (effects (font (size 1.27 1.27)) (justify right) hide)
     )
-  )
-  (global_label "HLIGHT1" (shape input) (at 163.83 46.99 180) (fields_autoplaced)
-    (effects (font (size 1.27 1.27)) (justify right))
-    (property "Intersheet References" "${INTERSHEET_REFS}" (id 0) (at 153.6759 46.9106 0)
-      (effects (font (size 1.27 1.27)) (justify right) hide)
-    )
-  )
-  (global_label "HLIGHT1" (shape input) (at 95.25 46.99 180) (fields_autoplaced)
-    (effects (font (size 1.27 1.27)) (justify right))
-    (property "Intersheet References" "${INTERSHEET_REFS}" (id 0) (at 85.0959 46.9106 0)
-      (effects (font (size 1.27 1.27)) (justify right) hide)
-    )
-  )
-  (symbol (lib_id "Device:R_Small") (at 59.69 46.99 90) (unit 1)
-    (in_bom yes) (on_board yes) (fields_autoplaced)
-    (property "Reference" "R14" (id 0) (at 59.69 40.64 90))
-    (property "Value" "100" (id 1) (at 59.69 43.18 90))
-    (property "Footprint" "UserLibrary:R_Axial_DIN0207_L6.3mm_D2.5mm_P10.16mm_Horizontal" (id 2) (at 59.69 46.99 0)
-      (effects (font (size 1.27 1.27)) hide)
-    )
-    (property "Datasheet" "~" (id 3) (at 59.69 46.99 0)
-      (effects (font (size 1.27 1.27)) hide)
-    )
-    (property "Nerokas link" "https://store.nerokas.co.ke/index.php?route=product/product&product_id=513&search=100+resistor&description=true" (id 4) (at 59.69 46.99 90)
-      (effects (font (size 1.27 1.27)) hide)
-    )
-    (pin "1")
-    (pin "2")
   )
   (symbol (lib_id "power:GND") (at 182.88 57.15 0) (unit 1)
@@
     )
     (pin "1")
-  )
-  (symbol (lib_id "Device:LED") (at 67.31 46.99 180) (unit 1)
-    (in_bom yes) (on_board yes) (fields_autoplaced)
-    (property "Reference" "D1" (id 0) (at 68.8975 39.37 0))
-    (property "Value" "LED" (id 1) (at 68.8975 41.91 0))
-    (property "Footprint" "LED_THT:LED_D5.0mm" (id 2) (at 67.31 46.99 0)
-      (effects (font (size 1.27 1.27)) hide)
-    )
-    (property "Datasheet" "~" (id 3) (at 67.31 46.99 0)
-      (effects (font (size 1.27 1.27)) hide)
-    )
-    (pin "1")
-    (pin "2")
-  )
-  (symbol (lib_id "power:GND") (at 74.93 57.15 0) (unit 1)
-    (in_bom yes) (on_board yes) (fields_autoplaced)
-    (property "Reference" "#PWR0143" (id 0) (at 74.93 63.5 0)
-      (effects (font (size 1.27 1.27)) hide)
-    )
-    (property "Value" "GND" (id 1) (at 74.93 62.23 0))
-    (property "Footprint" "" (id 2) (at 74.93 57.15 0)
-      (effects (font (size 1.27 1.27)) hide)
-    )
-    (property "Datasheet" "" (id 3) (at 74.93 57.15 0)
-      (effects (font (size 1.27 1.27)) hide)
-    )
-    (pin "1")
-  )
-  (symbol (lib_id "power:GND") (at 114.3 57.15 0) (unit 1)
-    (in_bom yes) (on_board yes) (fields_autoplaced)
-    (property "Reference" "#PWR0140" (id 0) (at 114.3 63.5 0)
-      (effects (font (size 1.27 1.27)) hide)
-    )
-    (property "Value" "GND" (id 1) (at 114.3 62.23 0))
-    (property "Footprint" "" (id 2) (at 114.3 57.15 0)
-      (effects (font (size 1.27 1.27)) hide)
-    )
-    (property "Datasheet" "" (id 3) (at 114.3 57.15 0)
-      (effects (font (size 1.27 1.27)) hide)
-    )
-    (pin "1")
-  )
-  (symbol (lib_id "Device:R_Small") (at 99.06 46.99 90) (unit 1)
-    (in_bom yes) (on_board yes) (fields_autoplaced)
-    (property "Reference" "R15" (id 0) (at 99.06 40.64 90))
-    (property "Value" "100" (id 1) (at 99.06 43.18 90))
-    (property "Footprint" "UserLibrary:R_Axial_DIN0207_L6.3mm_D2.5mm_P10.16mm_Horizontal" (id 2) (at 99.06 46.99 0)
-      (effects (font (size 1.27 1.27)) hide)
-    )
-    (property "Datasheet" "~" (id 3) (at 99.06 46.99 0)
-      (effects (font (size 1.27 1.27)) hide)
-    )
-    (property "Nerokas link" "https://store.nerokas.co.ke/index.php?route=product/product&product_id=513&search=100+resistor&description=true" (id 4) (at 99.06 46.99 90)
-      (effects (font (size 1.27 1.27)) hide)
-    )
-    (pin "1")
-    (pin "2")
   )
   (symbol (lib_id "Device:R_Small") (at 167.64 46.99 90) (unit 1)
@@
       (effects (font (size 1.27 1.27)) hide)
     )
-    (pin "1")
-    (pin "2")
-  )
-  (symbol (lib_id "Device:LED") (at 106.68 46.99 180) (unit 1)
-    (in_bom yes) (on_board yes) (fields_autoplaced)
-    (property "Reference" "D2" (id 0) (at 108.2675 39.37 0))
-    (property "Value" "LED" (id 1) (at 108.2675 41.91 0))
-    (property "Footprint" "LED_THT:LED_D5.0mm" (id 2) (at 106.68 46.99 0)
-      (effects (font (size 1.27 1.27)) hide)
-    )
-    (property "Datasheet" "~" (id 3) (at 106.68 46.99 0)
-      (effects (font (size 1.27 1.27)) hide)
-    )
-    (property "Nerokas link" "https://store.nerokas.co.ke/index.php?route=product/product&product_id=945&search=red+led+&description=true" (id 4) (at 106.68 46.99 0)
-      (effects (font (size 1.27 1.27)) hide)
-    )
