File: techweekpcb/sensors.kicad_sch (KiCad schematic)
At the start: 23 parts, among them J7 Conn_01x02_Male, J8 Conn_01x02_Male, Q2 IRLZ44N, Q3 IRLZ44N, Q4 IRLZ44N, Q5 IRLZ44N, Q6 IRLZ44N, Q7 IRLZ44N, U3 Ultrasonic, U4 Ultrasonic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

Commit message: Routing and Nerokas BOM
Parts:
- removed J7, J8: Conn_01x02_Male, Connector_PinHeader_2.54mm:PinHeader_1x02_P2.54mm_Vertical, symbol Connector:Conn_01x02_Male
- removed Q2, Q3, Q4, Q5, Q6, Q7: IRLZ44N, Package_TO_SOT_THT:TO-220-3_Vertical, symbol Transistor_FET:IRLZ44N
- removed R10, R11, R12, R13, R2, R3, R4, R5, R6, R7, R8, R9: 470, Resistor_THT:R_Axial_DIN0411_L9.9mm_D3.6mm_P12.70mm_Horizontal, symbol Device:R
- added R2, R4, R6: 1k, UserLibrary:R_Axial_DIN0207_L6.3mm_D2.5mm_P10.16mm_Horizontal, symbol Device:R_Small
- added R3, R5, R7: 2k, UserLibrary:R_Axial_DIN0207_L6.3mm_D2.5mm_P10.16mm_Horizontal, symbol Device:R_Small
Connections:
- net TRIG1 is gone; now on net ETRIG1: U3.2 (TRIG)
- net TRIG2 is gone; now on net ETRIG2: U4.2 (TRIG)
- net TRIG3 is gone; now on net ETRIG3: U5.2 (TRIG)
- net ECHO1: now also R2.1
- net ECHO2: now also R4.1
- net ECHO3: now also R6.1
- net EECHO1: now also R2.2, R3.1
- net EECHO2: now also R4.2, R5.1
- net EECHO3: now also R6.2, R7.1
- net GND: now also R3.2, R5.2, R7.2
Other:
- note removed: "+3v3 TRIG TO +5V"
- note removed: "+5V ECHO TO +3V3"
- note removed: "COMMS"
