File: techweekpcb/power.kicad_sch (KiCad schematic)
At the start: 10 parts, among them J1 Screw_Terminal_01x02, J2 Conn_01x02_Male, J3 Conn_01x02_Male, J4 Conn_01x02_Male, J5 Screw_Terminal_01x02, Q1 FQP27P06, U2 LM1084-5.0

Commit message: Routing and Nerokas BOM
Parts:
- removed J2, J3, J4: Conn_01x02_Male, Connector_PinHeader_2.54mm:PinHeader_1x02_P2.54mm_Vertical, symbol Connector:Conn_01x02_Male
- J1, J5: footprint TerminalBlock_Phoenix:TerminalBlock_Phoenix_MKDS-1,5-2-5.08_1x02_P5.08mm_Horizontal -> UserLibrary:TerminalBlock_Phoenix_MKDS-1,5-2-5.08_1x02_P5.08mm_Horizontal
- Q1: footprint Package_TO_SOT_THT:TO-220-3_Vertical -> UserLibrary:TO-220-3_Vertical
Changed lines of the file:
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@@
-    (stroke (width 0) (type default) (color 0 0 0 0))
-  )
-  (wire (pts (xy 133.35 109.22) (xy 138.43 109.22))
     (stroke (width 0) (type default) (color 0 0 0 0))
   )
@@
     (stroke (width 0) (type default) (color 0 0 0 0))
   )
-  (wire (pts (xy 138.43 109.22) (xy 138.43 111.76))
-    (stroke (width 0) (type default) (color 0 0 0 0))
-  )
   (wire (pts (xy 160.02 53.34) (xy 163.83 53.34))
     (stroke (width 0) (type default) (color 0 0 0 0))
@@
     (stroke (width 0) (type default) (color 0 0 0 0))
   )
-  (wire (pts (xy 156.21 107.95) (xy 163.83 107.95))
-    (stroke (width 0) (type default) (color 0 0 0 0))
-  )
   (polyline (pts (xy 129.54 31.75) (xy 129.54 77.47))
     (stroke (width 0) (type default) (color 0 0 0 0))
@@
     (stroke (width 0) (type default) (color 0 0 0 0))
   )
-  (wire (pts (xy 138.43 106.68) (xy 138.43 99.06))
-    (stroke (width 0) (type default) (color 0 0 0 0))
-  )
-  (wire (pts (xy 184.15 107.95) (xy 191.77 107.95))
-    (stroke (width 0) (type default) (color 0 0 0 0))
-  )
-  (wire (pts (xy 133.35 106.68) (xy 138.43 106.68))
-    (stroke (width 0) (type default) (color 0 0 0 0))
-  )
-  (wire (pts (xy 163.83 105.41) (xy 163.83 99.06))
-    (stroke (width 0) (type default) (color 0 0 0 0))
-  )
   (polyline (pts (xy 129.54 31.75) (xy 209.55 31.75))
     (stroke (width 0) (type default) (color 0 0 0 0))
@@
     (stroke (width 0) (type default) (color 0 0 0 0))
   )
-  (wire (pts (xy 184.15 105.41) (xy 191.77 105.41))
-    (stroke (width 0) (type default) (color 0 0 0 0))
-  )
-  (wire (pts (xy 163.83 107.95) (xy 163.83 111.76))
-    (stroke (width 0) (type default) (color 0 0 0 0))
-  )
   (polyline (pts (xy 207.01 142.24) (xy 269.24 142.24))
     (stroke (width 0) (type default) (color 0 0 0 0))
@@
     (stroke (width 0) (type default) (color 0 0 0 0))
   )
-  (wire (pts (xy 191.77 105.41) (xy 191.77 99.06))
-    (stroke (width 0) (type default) (color 0 0 0 0))
-  )
   (wire (pts (xy 59.69 107.95) (xy 63.5 107.95))
     (stroke (width 0) (type default) (color 0 0 0 0))
   )
-  (wire (pts (xy 191.77 107.95) (xy 191.77 111.76))
-    (stroke (width 0) (type default) (color 0 0 0 0))
-  )
   (wire (pts (xy 82.55 107.95) (xy 85.09 107.95))
-    (stroke (width 0) (type default) (color 0 0 0 0))
-  )
-  (wire (pts (xy 156.21 105.41) (xy 163.83 105.41))
     (stroke (width 0) (type default) (color 0 0 0 0))
   )
@@
     (pin "1")
   )
-  (symbol (lib_id "power:+5V") (at 163.83 99.06 0) (unit 1)
-    (in_bom yes) (on_board yes) (fields_autoplaced)
-    (property "Reference" "#PWR0118" (id 0) (at 163.83 102.87 0)
-      (effects (font (size 1.27 1.27)) hide)
-    )
-    (property "Value" "+5V" (id 1) (at 163.83 93.98 0))
-    (property "Footprint" "" (id 2) (at 163.83 99.06 0)
-      (effects (font (size 1.27 1.27)) hide)
-    )
-    (property "Datasheet" "" (id 3) (at 163.83 99.06 0)
-      (effects (font (size 1.27 1.27)) hide)
-    )
-    (pin "1")
-  )
   (symbol (lib_id "Connector:Screw_Terminal_01x02") (at 67.31 55.88 0) (unit 1)
     (in_bom yes) (on_board yes) (fields_autoplaced)
@@
       (effects (font (size 1.27 1.27)) (justify left) hide)
     )
-    (property "Footprint" "TerminalBlock_Phoenix:TerminalBlock_Phoenix_MKDS-1,5-2-5.08_1x02_P5.08mm_Horizontal" (id 2) (at 67.31 55.88 0)
+    (property "Footprint" "UserLibrary:TerminalBlock_Phoenix_MKDS-1,5-2-5.08_1x02_P5.08mm_Horizontal" (id 2) (at 67.31 55.88 0)
       (effects (font (size 1.27 1.27)) hide)
     )
@@
     (pin "3")
   )
-  (symbol (lib_id "power:+5V") (at 138.43 99.06 0) (unit 1)
-    (in_bom yes) (on_board yes) (fields_autoplaced)
-    (property "Reference" "#PWR0114" (id 0) (at 138.43 102.87 0)
-      (effects (font (size 1.27 1.27)) hide)
-    )
-    (property "Value" "+5V" (id 1) (at 138.43 93.98 0))
-    (property "Footprint" "" (id 2) (at 138.43 99.06 0)
-      (effects (font (size 1.27 1.27)) hide)
-    )
-    (property "Datasheet" "" (id 3) (at 138.43 99.06 0)
-      (effects (font (size 1.27 1.27)) hide)
-    )
-    (pin "1")
-  )
-  (symbol (lib_id "power:GND") (at 191.77 111.76 0) (unit 1)
-    (in_bom yes) (on_board yes) (fields_autoplaced)
-    (property "Reference" "#PWR0121" (id 0) (at 191.77 118.11 0)
-      (effects (font (size 1.27 1.27)) hide)
-    )
-    (property "Value" "GND" (id 1) (at 191.77 116.84 0))
-    (property "Footprint" "" (id 2) (at 191.77 111.76 0)
-      (effects (font (size 1.27 1.27)) hide)
-    )
-    (property "Datasheet" "" (id 3) (at 191.77 111.76 0)
-      (effects (font (size 1.27 1.27)) hide)
-    )
-    (pin "1")
-  )
   (symbol (lib_id "Device:C_Small") (at 85.09 110.49 0) (unit 1)
     (in_bom yes) (on_board yes) (fields_autoplaced)
@@
     (pin "1")
     (pin "2")
-  )
-  (symbol (lib_id "Connector:Conn_01x02_Male") (at 128.27 106.68 0) (unit 1)
-    (in_bom yes) (on_board yes) (fields_autoplaced)
-    (property "Reference" "J2" (id 0) (at 128.905 101.6 0))
-    (property "Value" "Conn_01x02_Male" (id 1) (at 128.905 104.14 0))
-    (property "Footprint" "Connector_PinHeader_2.54mm:PinHeader_1x02_P2.54mm_Vertical" (id 2) (at 128.27 106.68 0)
-      (effects (font (size 1.27 1.27)) hide)
-    )
-    (property "Datasheet" "~" (id 3) (at 128.27 106.68 0)
-      (effects (font (size 1.27 1.27)) hide)
-    )
-    (property "Nerokas link" "https://store.nerokas.co.ke/index.php?route=product/product&product_id=955&search=Header+male&description=true" (id 4) (at 128.27 106.68 0)
-      (effects (font (size 1.27 1.27)) hide)
-    )
-    (pin "1")
-    (pin "2")
-  )
-  (symbol (lib_id "power:GND") (at 163.83 111.76 0) (unit 1)
-    (in_bom yes) (on_board yes) (fields_autoplaced)
-    (property "Reference" "#PWR0119" (id 0) (at 163.83 118.11 0)
-      (effects (font (size 1.27 1.27)) hide)
-    )
-    (property "Value" "GND" (id 1) (at 163.83 116.84 0))
-    (property "Footprint" "" (id 2) (at 163.83 111.76 0)
-      (effects (font (size 1.27 1.27)) hide)
-    )
-    (property "Datasheet" "" (id 3) (at 163.83 111.76 0)
-      (effects (font (size 1.27 1.27)) hide)
-    )
-    (pin "1")
   )
   (symbol (lib_id "Transistor_FET:AO3401A") (at 168.91 55.88 90) (unit 1)
@@
     (property "Reference" "Q1" (id 0) (at 168.91 45.72 90))
     (property "Value" "FQP27P06" (id 1) (at 168.91 48.26 90))
-    (property "Footprint" "Package_TO_SOT_THT:TO-220-3_Vertical" (id 2) (at 170.815 50.8 0)
+    (property "Footprint" "UserLibrary:TO-220-3_Vertical" (id 2) (at 170.815 50.8 0)
       (effects (font (size 1.27 1.27) italic) (justify left) hide)
     )
@@
     (pin "3")
   )
-  (symbol (lib_id "power:+3V3") (at 191.77 99.06 0) (unit 1)
-    (in_bom yes) (on_board yes) (fields_autoplaced)
-    (property "Reference" "#PWR0120" (id 0) (at 191.77 102.87 0)
-      (effects (font (size 1.27 1.27)) hide)
-    )
-    (property "Value" "+3V3" (id 1) (at 191.77 93.98 0))
-    (property "Footprint" "" (id 2) (at 191.77 99.06 0)
-      (effects (font (size 1.27 1.27)) hide)
-    )
-    (property "Datasheet" "" (id 3) (at 191.77 99.06 0)
-      (effects (font (size 1.27 1.27)) hide)
-    )
-    (pin "1")
-  )
   (symbol (lib_id "power:+12V") (at 177.8 48.26 0) (unit 1)
     (in_bom yes) (on_board yes) (fields_autoplaced)
@@
     (pin "2")
   )
-  (symbol (lib_id "Connector:Conn_01x02_Male") (at 151.13 105.41 0) (unit 1)
-    (in_bom yes) (on_board yes) (fields_autoplaced)
-    (property "Reference" "J3" (id 0) (at 151.765 100.33 0))
-    (property "Value" "Conn_01x02_Male" (id 1) (at 151.765 102.87 0))
-    (property "Footprint" "Connector_PinHeader_2.54mm:PinHeader_1x02_P2.54mm_Vertical" (id 2) (at 151.13 105.41 0)
-      (effects (font (size 1.27 1.27)) hide)
-    )
-    (property "Datasheet" "~" (id 3) (at 151.13 105.41 0)
-      (effects (font (size 1.27 1.27)) hide)
-    )
-    (property "Nerokas link" "https://store.nerokas.co.ke/index.php?route=product/product&product_id=955&search=Header+male&description=true" (id 4) (at 151.13 105.41 0)
-      (effects (font (size 1.27 1.27)) hide)
-    )
-    (pin "1")
-    (pin "2")
-  )
-  (symbol (lib_id "power:GND") (at 138.43 111.76 0) (unit 1)
-    (in_bom yes) (on_board yes) (fields_autoplaced)
-    (property "Reference" "#PWR0115" (id 0) (at 138.43 118.11 0)
-      (effects (font (size 1.27 1.27)) hide)
-    )
-    (property "Value" "GND" (id 1) (at 138.43 116.84 0))
-    (property "Footprint" "" (id 2) (at 138.43 111.76 0)
-      (effects (font (size 1.27 1.27)) hide)
-    )
-    (property "Datasheet" "" (id 3) (at 138.43 111.76 0)
-      (effects (font (size 1.27 1.27)) hide)
-    )
-    (pin "1")
-  )
-  (symbol (lib_id "Connector:Conn_01x02_Male") (at 179.07 105.41 0) (unit 1)
-    (in_bom yes) (on_board yes) (fields_autoplaced)
-    (property "Reference" "J4" (id 0) (at 179.705 100.33 0))
-    (property "Value" "Conn_01x02_Male" (id 1) (at 179.705 102.87 0))
-    (property "Footprint" "Connector_PinHeader_2.54mm:PinHeader_1x02_P2.54mm_Vertical" (id 2) (at 179.07 105.41 0)
-      (effects (font (size 1.27 1.27)) hide)
-    )
-    (property "Datasheet" "~" (id 3) (at 179.07 105.41 0)
-      (effects (font (size 1.27 1.27)) hide)
-    )
-    (property "Nerokas link" "https://store.nerokas.co.ke/index.php?route=product/product&product_id=955&search=Header+male&description=true" (id 4) (at 179.07 105.41 0)
-      (effects (font (size 1.27 1.27)) hide)
-    )
-    (pin "1")
-    (pin "2")
-  )
   (symbol (lib_id "power:GND") (at 168.91 68.58 0) (unit 1)
     (in_bom yes) (on_board yes) (fields_autoplaced)
@@
       (effects (font (size 1.27 1.27)) (justify left) hide)
     )
-    (property "Footprint" "TerminalBlock_Phoenix:TerminalBlock_Phoenix_MKDS-1,5-2-5.08_1x02_P5.08mm_Horizontal" (id 2) (at 234.95 104.14 0)
-      (effects (font (size 1.27 1.27)) hide)
-    )
+    (property "Footprint" "UserLibrary:TerminalBlock_Phoenix_MKDS-1,5-2-5.08_1x02_P5.08mm_Horizontal" (id 2) (at 234.95 104.14 0)
+      (effects (font (size 1.27 1.27)) hide)
+    )

Commit message: Updating BOM
Parts:
- Q1, U2: now left out of the parts list
Other:
- moved on the sheet: J5
Changed lines of the file:
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@@
     (stroke (width 0) (type default) (color 0 0 0 0))
   )
-  (polyline (pts (xy 269.24 142.24) (xy 269.24 82.55))
+  (polyline (pts (xy 168.91 142.24) (xy 168.91 82.55))
     (stroke (width 0) (type default) (color 0 0 0 0))
   )
@@
     (stroke (width 0) (type default) (color 0 0 0 0))
   )
-  (polyline (pts (xy 207.01 82.55) (xy 269.24 82.55))
+  (polyline (pts (xy 106.68 82.55) (xy 168.91 82.55))
     (stroke (width 0) (type default) (color 0 0 0 0))
   )
@@
     (stroke (width 0) (type default) (color 0 0 0 0))
   )
-  (wire (pts (xy 229.87 109.22) (xy 229.87 106.68))
+  (wire (pts (xy 129.54 109.22) (xy 129.54 106.68))
     (stroke (width 0) (type default) (color 0 0 0 0))
   )
@@
     (stroke (width 0) (type default) (color 0 0 0 0))
   )
-  (wire (pts (xy 229.87 101.6) (xy 229.87 104.14))
+  (wire (pts (xy 129.54 101.6) (xy 129.54 104.14))
     (stroke (width 0) (type default) (color 0 0 0 0))
   )
@@
     (stroke (width 0) (type default) (color 0 0 0 0))
   )
-  (polyline (pts (xy 207.01 82.55) (xy 207.01 142.24))
-    (stroke (width 0) (type default) (color 0 0 0 0))
-  )
-  (polyline (pts (xy 207.01 142.24) (xy 269.24 142.24))
+  (polyline (pts (xy 106.68 82.55) (xy 106.68 142.24))
+    (stroke (width 0) (type default) (color 0 0 0 0))
+  )
+  (polyline (pts (xy 106.68 142.24) (xy 168.91 142.24))
     (stroke (width 0) (type default) (color 0 0 0 0))
   )
@@
     (effects (font (size 4 4)) (justify left bottom))
   )
-  (text "DRIVER PWR\n" (at 218.44 91.44 0)
+  (text "DRIVER PWR\n" (at 118.11 91.44 0)
     (effects (font (size 4 4)) (justify left bottom))
   )
@@
   )
   (symbol (lib_id "Regulator_Linear:LM1084-5.0") (at 74.93 107.95 0) (unit 1)
-    (in_bom yes) (on_board yes)
+    (in_bom no) (on_board yes)
     (property "Reference" "U2" (id 0) (at 74.93 91.44 0))
     (property "Value" "LM1084-5.0" (id 1) (at 74.93 93.98 0))
@@
   )
   (symbol (lib_id "Transistor_FET:AO3401A") (at 168.91 55.88 90) (unit 1)
-    (in_bom yes) (on_board yes) (fields_autoplaced)
+    (in_bom no) (on_board yes) (fields_autoplaced)
     (property "Reference" "Q1" (id 0) (at 168.91 45.72 90))
     (property "Value" "FQP27P06" (id 1) (at 168.91 48.26 90))
@@
     (pin "1")
   )
-  (symbol (lib_id "power:+12V") (at 229.87 101.6 0) (unit 1)
-    (in_bom yes) (on_board yes) (fields_autoplaced)
-    (property "Reference" "#PWR0117" (id 0) (at 229.87 105.41 0)
-      (effects (font (size 1.27 1.27)) hide)
-    )
-    (property "Value" "+12V" (id 1) (at 229.87 96.52 0))
-    (property "Footprint" "" (id 2) (at 229.87 101.6 0)
-      (effects (font (size 1.27 1.27)) hide)
-    )
-    (property "Datasheet" "" (id 3) (at 229.87 101.6 0)
+  (symbol (lib_id "power:+12V") (at 129.54 101.6 0) (unit 1)
+    (in_bom yes) (on_board yes) (fields_autoplaced)
+    (property "Reference" "#PWR0117" (id 0) (at 129.54 105.41 0)
+      (effects (font (size 1.27 1.27)) hide)
+    )
+    (property "Value" "+12V" (id 1) (at 129.54 96.52 0))
+    (property "Footprint" "" (id 2) (at 129.54 101.6 0)
+      (effects (font (size 1.27 1.27)) hide)
+    )
+    (property "Datasheet" "" (id 3) (at 129.54 101.6 0)
       (effects (font (size 1.27 1.27)) hide)
     )
@@
     (pin "1")
   )
-  (symbol (lib_id "Connector:Screw_Terminal_01x02") (at 234.95 104.14 0) (unit 1)
-    (in_bom yes) (on_board yes) (fields_autoplaced)
-    (property "Reference" "J5" (id 0) (at 237.49 105.4099 0)
-      (effects (font (size 1.27 1.27)) (justify left))
-    )
-    (property "Value" "Screw_Terminal_01x02" (id 1) (at 237.49 106.6799 0)
+  (symbol (lib_id "Connector:Screw_Terminal_01x02") (at 134.62 104.14 0) (unit 1)
+    (in_bom yes) (on_board yes) (fields_autoplaced)
+    (property "Reference" "J5" (id 0) (at 137.16 105.4099 0)
+      (effects (font (size 1.27 1.27)) (justify left))
+    )
+    (property "Value" "Screw_Terminal_01x02" (id 1) (at 137.16 106.6799 0)
       (effects (font (size 1.27 1.27)) (justify left) hide)
     )
-    (property "Footprint" "UserLibrary:TerminalBlock_Phoenix_MKDS-1,5-2-5.08_1x02_P5.08mm_Horizontal" (id 2) (at 234.95 104.14 0)
-      (effects (font (size 1.27 1.27)) hide)
-    )
-    (property "Datasheet" "~" (id 3) (at 234.95 104.14 0)
-      (effects (font (size 1.27 1.27)) hide)
-    )
-    (property "Nerokas link" "https://store.nerokas.co.ke/index.php?route=product/product&product_id=2056" (id 4) (at 234.95 104.14 0)
-      (effects (font (size 1.27 1.27)) hide)
-    )
-    (pin "1")
-    (pin "2")
-  )
-  (symbol (lib_id "power:GND") (at 229.87 109.22 0) (unit 1)
-    (in_bom yes) (on_board yes) (fields_autoplaced)
-    (property "Reference" "#PWR0116" (id 0) (at 229.87 115.57 0)
-      (effects (font (size 1.27 1.27)) hide)
-    )
-    (property "Value" "GND" (id 1) (at 229.87 114.3 0))
-    (property "Footprint" "" (id 2) (at 229.87 109.22 0)
-      (effects (font (size 1.27 1.27)) hide)
-    )
-    (property "Datasheet" "" (id 3) (at 229.87 109.22 0)
+    (property "Footprint" "UserLibrary:TerminalBlock_Phoenix_MKDS-1,5-2-5.08_1x02_P5.08mm_Horizontal" (id 2) (at 134.62 104.14 0)
+      (effects (font (size 1.27 1.27)) hide)
+    )
+    (property "Datasheet" "~" (id 3) (at 134.62 104.14 0)
+      (effects (font (size 1.27 1.27)) hide)
+    )
+    (property "Nerokas link" "https://store.nerokas.co.ke/index.php?route=product/product&product_id=2056" (id 4) (at 134.62 104.14 0)
+      (effects (font (size 1.27 1.27)) hide)
+    )
+    (pin "1")
+    (pin "2")
+  )
+  (symbol (lib_id "power:GND") (at 129.54 109.22 0) (unit 1)
+    (in_bom yes) (on_board yes) (fields_autoplaced)
+    (property "Reference" "#PWR0116" (id 0) (at 129.54 115.57 0)
+      (effects (font (size 1.27 1.27)) hide)
+    )
+    (property "Value" "GND" (id 1) (at 129.54 114.3 0))
+    (property "Footprint" "" (id 2) (at 129.54 109.22 0)
+      (effects (font (size 1.27 1.27)) hide)
+    )
+    (property "Datasheet" "" (id 3) (at 129.54 109.22 0)
       (effects (font (size 1.27 1.27)) hide)
     )
@@
     (pin "1")
   )
+  (sheet_instances
+    (path "/" (page "1"))
+  )
+  (symbol_instances
+    (path "/f31670be-b100-4560-81a7-697f3f095318"
+      (reference "#PWR0104") (unit 1) (value "GND") (footprint "")
+    )
+    (path "/0cb1d0b5-981b-4e4a-87b8-cad3d4ca87f7"
+      (reference "#PWR0105") (unit 1) (value "+5V") (footprint "")
+    )
+    (path "/b68dbaa1-5d3d-40c2-8fb1-df43a463fa0a"
+      (reference "#PWR0106") (unit 1) (value "GND") (footprint "")
+    )
+    (path "/d9d858e8-ed66-48b3-ab4d-c67fcb6db6b1"
+      (reference "#PWR0107") (unit 1) (value "GND") (footprint "")
+    )
+    (path "/015b1c8f-68b5-4492-afed-ea89b5fa0da2"
+      (reference "#PWR0108") (unit 1) (value "+12V") (footprint "")
+    )
+    (path "/d8b647f8-124e-4eda-a5be-c64e3a6d4ace"
+      (reference "#PWR0109") (unit 1) (value "+12P") (footprint "")
+    )
+    (path "/b748843b-4c8f-4900-8f10-00b252ab59d2"
+      (reference "#PWR0110") (unit 1) (value "GND") (footprint "")
+    )
+    (path "/ae5d0342-9eb3-40eb-ac59-0260460d2f58"
+      (reference "#PWR0111") (unit 1) (value "GND") (footprint "")
+    )
+    (path "/6e3e0bde-ef70-4b23-b270-2fb10325b77f"
+      (reference "#PWR0112") (unit 1) (value "+12V") (footprint "")
+    )
+    (path "/e7ff73a9-920a-42dd-8798-cf5d24d7a0ca"
+      (reference "#PWR0113") (unit 1) (value "+12P") (footprint "")
+    )
+    (path "/e354a026-c1cc-4c96-ae01-e7e75cc842f5"
+      (reference "#PWR0116") (unit 1) (value "GND") (footprint "")
+    )
+    (path "/cf7f5296-1365-464c-b3c3-186906fb4dc1"
+      (reference "#PWR0117") (unit 1) (value "+12V") (footprint "")
+    )
+    (path "/0aa7af07-8a79-4608-8854-631ee897834b"
+      (reference "C1") (unit 1) (value "10uF") (footprint "UserLibrary:CP_Radial_D5.0mm_P2.50mm")
+    )
+    (path "/46541204-adf3-48ab-8d31-e267274fde4a"
+      (reference "C2") (unit 1) (value "10uF") (footprint "UserLibrary:CP_Radial_D5.0mm_P2.50mm")
+    )
+    (path "/0a5a1cf7-5bf0-45bb-8006-a1ec23c250c1"
+      (reference "J1") (unit 1) (value "Screw_Terminal_01x02") (footprint "UserLibrary:TerminalBlock_Phoenix_MKDS-1,5-2-5.08_1x02_P5.08mm_Horizontal")
+    )
+    (path "/db47a2f6-972e-40d2-ba12-c0402958a215"
+      (reference "J5") (unit 1) (value "Screw_Terminal_01x02") (footprint "UserLibrary:TerminalBlock_Phoenix_MKDS-1,5-2-5.08_1x02_P5.08mm_Horizontal")
+    )
+    (path "/597f6f6a-e1c9-4d0a-8ab5-49d7236018ab"
+      (reference "Q1") (unit 1) (value "FQP27P06") (footprint "UserLibrary:TO-220-3_Vertical")
+    )
+    (path "/7cd91072-e687-4422-83db-665db3601aba"
+      (reference "R1") (unit 1) (value "1.1k") (footprint "Resistor_THT:R_Axial_DIN0207_L6.3mm_D2.5mm_P10.16mm_Horizontal")
+    )
+    (path "/0f72e55d-9589-4792-a23e-a3b6a0476e5a"
+      (reference "U2") (unit 1) (value "LM1084-5.0") (footprint "UserLibrary:TO-220-3_Vertical")
+    )
+  )
 )
