File: techweekpcb/techweekpcb.kicad_sch (KiCad schematic)
At the start: 1 part, among them U1 ESP32-S

Commit message: Routing and Nerokas BOM
Parts:
- added H1, H2, H3, H4: MountingHole, MountingHole:MountingHole_2.5mm, symbol Mechanical:MountingHole
Connections:
- net EECHO2: now also U1.31 (P14); no longer U1.11 (P18), U1.32 (P12)
- net ENA: now also U1.18 (P23); no longer U1.12 (P19)
- net ETRIG2: now also U1.32 (P12); no longer U1.10 (P5), U1.34 (P13)
- net GND: now also U1.13 (GND), U1.33 (GND)
- net IN1: now also U1.12 (P19); no longer U1.18 (P23)
- net IN2: now also U1.11 (P18); no longer U1.26 (P32)
- net EECHO3: now reaches U1.30 (P27)
- net RLIGHT4: now reaches U1.8 (P16)
- net RLIGHT3: now reaches U1.9 (P17)
- net +3V3 renamed +3.3V
- new net ETRIG3: U1.34 (P13)
- no-connect marks 2 -> 3

Commit message: Updating BOM
Parts:
- U1: now left out of the parts list
Changed lines of the file:
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@@
   )
   (symbol (lib_id "Userlibrary:ESP32-S") (at 205.74 83.82 0) (unit 1)
-    (in_bom yes) (on_board yes) (fields_autoplaced)
+    (in_bom no) (on_board yes) (fields_autoplaced)
     (property "Reference" "U1" (id 0) (at 205.74 53.34 0))
     (property "Value" "ESP32-S" (id 1) (at 205.74 55.88 0))
